Commit message: add color

File: my_robot/urdf/my_robot.xacro (robot description, xacro)
@@ -30,22 +30,4 @@
         <box size=".4 .25 .1"/>
       </geometry>
-      <material name="red">
-        <color rgba="1 0 0 1"/>
-      </material>
-    </visual>
-    <collision name='head_collision'>
-      <origin xyz="0.2 0 0" rpy=" 0 0 0"/>
-      <geometry>
-        <cylinder radius="0.125" length="0.1"/>
-      </geometry>
-    </collision>
-    <visual name='head_visual'>
-      <origin xyz="0.2 0 0" rpy=" 0 0 0"/>
-      <geometry>
-        <cylinder radius="0.125" length="0.1"/>
-      </geometry>
-      <material name="red">
-        <color rgba="1 0 0 1"/>
-      </material>
     </visual>
     <collision name='back_caster_collision'>
@@ -60,24 +42,39 @@
         <sphere radius="0.06"/>
       </geometry>
-      <material name="orange">
-        <color rgba="1 0.5 0 1"/>
-      </material>
-    </visual>
-    <!-- <collision name='front_caster_collision'>
-      <origin xyz="0.2 0 -0.05" rpy=" 0 0 0"/>
-      <geometry>
-        <sphere radius="0.0599"/>
-      </geometry>
-    </collision> -->
-    <!-- <visual name='front_caster_visual'>
-      <origin xyz="0.2 0 -0.05" rpy=" 0 0 0"/>
-      <geometry>
-        <sphere radius="0.06"/>
-      </geometry>
-      <material name="orange">
-        <color rgba="1 0.5 0 1"/>
-      </material>
-    </visual> -->
-  </link>
+    </visual>
+  </link>
+  <gazebo reference="chassis">
+    <material>Gazebo/Green</material>
+  </gazebo>
+  <joint type="fixed" name="head_joint">
+    <origin xyz="0.2 0 0" rpy="0 0 0"/>
+    <child link="head"/>
+    <parent link="chassis"/>
+  </joint>
+  <link name='head'>
+    <inertial>
+      <mass value="10.0"/>
+      <inertia
+          ixx="0.1" ixy="0" ixz="0"
+          iyy="0.1" iyz="0"
+          izz="0.1"
+      />
+    </inertial>
+    <collision name='head_collision'>
+      <origin xyz="0 0 0" rpy=" 0 0 0"/>
+      <geometry>
+        <cylinder radius="0.125" length="0.1"/>
+      </geometry>
+    </collision>
+    <visual name='head_visual'>
+      <origin xyz="0 0 0" rpy=" 0 0 0"/>
+      <geometry>
+        <cylinder radius="0.125" length="0.1"/>
+      </geometry>
+    </visual>
+  </link>
+  <gazebo reference="head">
+    <material>Gazebo/Green</material>
+  </gazebo>
   <joint type="continuous" name="left_wheel_hinge">
     <origin xyz="0.1 0.15 0" rpy="0 0 0"/>
@@ -85,12 +82,10 @@
     <parent link="chassis"/>
     <axis xyz="0 1 0" rpy="0 0 0"/>
-    <limit effort="10000" velocity="1000"/>
+    <!-- <limit effort="10000" velocity="1000"/> -->
     <dynamics damping="1.0" friction="1.0"/>
   </joint>
   <link name='left_wheel'>
-    <!-- <pose>0 0 0.1 0 0 0</pose> -->
     <inertial>
       <mass value="5.0"/>
-      <!-- <origin xyz="0.0 0 0" rpy=" 0 1.5707 1.5707"/> -->
       <inertia
           ixx="0.1" ixy="0" ixz="0"
@@ -110,9 +105,9 @@
         <cylinder radius="0.11" length= "0.05"/>
       </geometry>
-      <material name="lw_yellow">
-        <color rgba="1 1 0 1"/>
-      </material>
-    </visual>
-  </link>
+    </visual>
+  </link>
+  <gazebo reference="left_wheel">
+    <material>Gazebo/Yellow</material>
+  </gazebo>
   <joint type="continuous" name="right_wheel_hinge">
     <origin xyz="0.1 -0.15 0" rpy="0 0 0"/>
@@ -120,12 +115,10 @@
     <parent link="chassis"/>
     <axis xyz="0 1 0" rpy="0 0 0"/>
-    <limit effort="10000" velocity="1000"/>
+    <!-- <limit effort="10000" velocity="1000"/> -->
     <dynamics damping="1.0" friction="1.0"/>
   </joint>
   <link name='right_wheel'>
-    <!-- <pose>0 0 0.1 0 0 0</pose> -->
     <inertial>
       <mass value="5.0"/>
-      <!-- <origin xyz="0.0 0 0" rpy=" 0 1.5707 1.5707"/> -->
       <inertia
           ixx="0.1" ixy="0" ixz="0"
@@ -145,9 +138,9 @@
         <cylinder radius="0.11" length= "0.05"/>
       </geometry>
-      <material name="rw_yellow">
-        <color rgba="1 1 0 1"/>
-      </material>
-    </visual>
-  </link>
+    </visual>
+  </link>
+  <gazebo reference="right_wheel">
+    <material>Gazebo/Yellow</material>
+  </gazebo>
   <joint type="fixed" name="camera_joint">
     <origin xyz="0.33 0 0" rpy="0 0 0"/>
@@ -159,5 +152,4 @@
     <inertial>
       <mass value="0.1"/>
-      <!-- <origin xyz="0.0 0 0" rpy=" 0 0 0"/> -->
       <inertia
           ixx="1e-6" ixy="0" ixz="0"
@@ -177,9 +169,9 @@
         <box size="0.05 0.05 0.05"/>
       </geometry>
-      <material name="green">
-        <color rgba="0 1 0 1"/>
-      </material>
-    </visual>
-  </link>
+    </visual>
+  </link>
+  <gazebo reference="camera">
+    <material>Gazebo/Red</material>
+  </gazebo>
   <joint type="fixed" name="hokuyo_joint">
     <origin xyz="0.27 0 0.08" rpy="0 0 0"/>
@@ -191,5 +183,4 @@
     <inertial>
       <mass value="1e-5"/>
-      <!-- <origin xyz="0.0 0 0" rpy=" 0 0 0"/> -->
       <inertia
           ixx="1e-6" ixy="0" ixz="0"

Commit message: add some new attempt.

File: my_robot/urdf/my_robot.xacro (robot description, xacro)
@@ -54,5 +54,5 @@
   <link name='head'>
     <inertial>
-      <mass value="10.0"/>
+      <mass value="0.01"/>
       <inertia
           ixx="0.1" ixy="0" ixz="0"

Commit message: Update RGBD sensor

File: my_robot/urdf/my_robot.xacro (robot description, xacro)
@@ -174,4 +174,11 @@
     <material>Gazebo/Red</material>
   </gazebo>
+  <joint name="camera_optical_joint" type="fixed">
+    <origin xyz="0 0 0" rpy="-1.5707 0 -1.5707"/>
+    <parent link="camera"/>
+    <child link="camera_d"/>
+  </joint>
+  <link name="camera_d">
+  </link>
   <joint type="fixed" name="hokuyo_joint">
     <origin xyz="0.27 0 0.08" rpy="0 0 0"/>

Commit message: clean up the repo for the map my world project

File: my_robot/urdf/my_robot.xacro (robot description, xacro)
@@ -22,5 +22,5 @@
       <origin xyz="0 0 0" rpy=" 0 0 0"/>
       <geometry>
-        <box size=".4 .25 .1"/>
+        <box size=".4 .2 .1"/>
       </geometry>
     </collision>
@@ -28,17 +28,29 @@
       <origin xyz="0 0 0" rpy=" 0 0 0"/>
       <geometry>
-        <box size=".4 .25 .1"/>
-      </geometry>
-    </visual>
+        <box size=".4 .2 .1"/>
+      </geometry>
+    </visual>
+    <collision name='front_caster_collision'>
+      <origin xyz="0.15 0 -0.05" rpy=" 0 0 0"/>
+        <geometry>
+          <sphere radius="0.0499"/>
+        </geometry>
+      </collision>
+      <visual name='front_caster_visual'>
+        <origin xyz="0.15 0 -0.05" rpy=" 0 0 0"/>
+        <geometry>
+          <sphere radius="0.05"/>
+        </geometry>
+      </visual>
     <collision name='back_caster_collision'>
-      <origin xyz="-0.12 0 -0.05" rpy=" 0 0 0"/>
-      <geometry>
-        <sphere radius="0.0599"/>
+      <origin xyz="-0.15 0 -0.05" rpy=" 0 0 0"/>
+      <geometry>
+        <sphere radius="0.0499"/>
       </geometry>
     </collision>
     <visual name='back_caster_visual'>
-      <origin xyz="-0.12 0 -0.05" rpy=" 0 0 0"/>
-      <geometry>
-        <sphere radius="0.06"/>
+      <origin xyz="-0.15 0 -0.05" rpy=" 0 0 0"/>
+      <geometry>
+        <sphere radius="0.05"/>
       </geometry>
     </visual>
@@ -47,5 +59,5 @@
     <material>Gazebo/Green</material>
   </gazebo>
-  <joint type="fixed" name="head_joint">
+  <!-- <joint type="fixed" name="head_joint">
     <origin xyz="0.2 0 0" rpy="0 0 0"/>
     <child link="head"/>
@@ -76,11 +88,11 @@
   <gazebo reference="head">
     <material>Gazebo/Green</material>
-  </gazebo>
+  </gazebo> -->
   <joint type="continuous" name="left_wheel_hinge">
-    <origin xyz="0.1 0.15 0" rpy="0 0 0"/>
+    <origin xyz="0.0 0.15 0" rpy="0 0 0"/>
     <child link="left_wheel"/>
     <parent link="chassis"/>
     <axis xyz="0 1 0" rpy="0 0 0"/>
-    <!-- <limit effort="10000" velocity="1000"/> -->
+    <limit effort="10000" velocity="1000"/>
     <dynamics damping="1.0" friction="1.0"/>
   </joint>
@@ -97,5 +109,5 @@
       <origin xyz="0 0 0" rpy=" 0 1.5707 1.5707"/>
       <geometry>
-        <cylinder radius="0.11" length= "0.05"/>
+        <cylinder radius="0.1" length= "0.05"/>
       </geometry>
     </collision>
@@ -103,5 +115,5 @@
       <origin xyz="0 0 0" rpy=" 0 1.5707 1.5707"/>
       <geometry>
-        <cylinder radius="0.11" length= "0.05"/>
+        <cylinder radius="0.1" length= "0.05"/>
       </geometry>
     </visual>
@@ -111,9 +123,9 @@
   </gazebo>
   <joint type="continuous" name="right_wheel_hinge">
-    <origin xyz="0.1 -0.15 0" rpy="0 0 0"/>
+    <origin xyz="0.0 -0.15 0" rpy="0 0 0"/>
     <child link="right_wheel"/>
     <parent link="chassis"/>
     <axis xyz="0 1 0" rpy="0 0 0"/>
-    <!-- <limit effort="10000" velocity="1000"/> -->
+    <limit effort="10000" velocity="1000"/>
     <dynamics damping="1.0" friction="1.0"/>
   </joint>
@@ -130,5 +142,5 @@
       <origin xyz="0 0 0" rpy=" 0 1.5707 1.5707"/>
       <geometry>
-        <cylinder radius="0.11" length= "0.05"/>
+        <cylinder radius="0.1" length= "0.05"/>
       </geometry>
     </collision>
@@ -136,5 +148,5 @@
       <origin xyz="0 0 0" rpy=" 0 1.5707 1.5707"/>
       <geometry>
-        <cylinder radius="0.11" length= "0.05"/>
+        <cylinder radius="0.1" length= "0.05"/>
       </geometry>
     </visual>
@@ -144,5 +156,5 @@
   </gazebo>
   <joint type="fixed" name="camera_joint">
-    <origin xyz="0.33 0 0" rpy="0 0 0"/>
+    <origin xyz="0.2 0 0" rpy="0 0 0"/>
     <child link="camera"/>
     <parent link="chassis"/>
@@ -182,5 +194,5 @@
   </link>
   <joint type="fixed" name="hokuyo_joint">
-    <origin xyz="0.27 0 0.08" rpy="0 0 0"/>
+    <origin xyz="0.15 0 0.1" rpy="0 0 0"/>
     <child link="hokuyo"/>
     <parent link="chassis"/>
